File: Fuente/Fuente.kicad_sch (KiCad schematic)
At the start: 1 part, among them U1 SG3525

Commit message: testestest
Parts:
- added C1, C2: C, symbol Device:C
- added R1, R2, R3, R4, R6, R7, R8: R, symbol Device:R
- added RV1: R_Potentiometer, symbol Device:R_Potentiometer
Connections:
- net at U1.1 (INV): now also R4.1, R6.2
- net at U1.10 (SD): now also C1.1, R7.2
- net PWM: now reaches U1.11 (OUTA)
- net GND: now reaches U1.12 (GND)
- net GND: now also C1.2, C2.2, R2.2, R7.1, R8.2, RV1.3
- net 15V: now reaches U1.15 (VIN)
- net at U1.16 (REF): now also R1.1
- net at U1.2 (NI): now also R3.2, RV1.1
- net at U1.5 (CT): now also U1.7 (DISCH), C2.1
- net at U1.6 (RT): now also R8.1
- net at U1.9 (COMP): now also R4.2
- new net: R1.2, R2.1, R3.1
- new net: R6.1, RV1.2
- no-connect marks 0 -> 3
